File: shark1by3.kicad_sch (KiCad schematic)
At the start: 0 parts

Commit message: plan schema
Parts:
- added C1, C2: 22pF, symbol Device:C_Small
- added C3, C4, C5, C6: .1uF, symbol Device:C_Small
- added C7: 10uF, symbol Device:C_Small
- added C8: 1uF, symbol Device:C_Small
- added D1, D2, D3: D, symbol Device:D_Small
- added F1: 500mA, symbol Device:Polyfuse_Small
- added J1: AVR-ISP-6, symbol Connector:AVR-ISP-6
- added MX1: Z, symbol MX_Alps_Hybrid:MX-NoLED
- added MX2: X, symbol MX_Alps_Hybrid:MX-NoLED
- added MX3: C, symbol MX_Alps_Hybrid:MX-NoLED
- added R1, R6: 10k, symbol Device:R_Small
- added R2, R3: 22, symbol Device:R_Small
- added R4, R5: 5.1k, symbol Device:R_Small
- added SW1: SW_Push_Reset, symbol local:SW_SKQG
- added U1: PRTR5V0U2X, symbol random-keyboard-parts:PRTR5V0U2X
- added U2: ATmega32U4-A, Package_QFP:TQFP-44_10x10mm_P0.8mm, symbol MCU_Microchip_ATmega:ATmega32U4-A
- added USB1: HRO-TYPE-C-31-M-12, symbol Type-C:HRO-TYPE-C-31-M-12
- added X1: 16MHz, symbol Device:Crystal_GND24_Small
Connections:
- new net: D1.2 (A), MX1.2 (ROW)
- new net: R6.1, U2.33 (~{HWB}/PE2)
- new net: C8.2, U2.6 (UCAP)
- new net: R4.1, USB1.10 (CC2)
- new net: R5.1, USB1.4 (CC1)
- new net: R2.1, U1.3 (IO2), USB1.5 (DN2), USB1.7 (DN1)
- new net: R3.1, U1.2 (IO1), USB1.6 (DP1), USB1.8 (DP2)
- new net: D3.2 (A), MX3.2 (ROW)
- new net: D2.2 (A), MX2.2 (ROW)
- new net +5V: C3.1, C4.1, C5.1, C6.1, C7.1, F1.2, J1.2 (VCC), R1.1, U2.14 (VCC), U2.2 (UVCC), U2.24 (AVCC), U2.34 (VCC), U2.44 (AVCC), U2.7 (VBUS)
- new net D+: R3.2, U2.4 (D+)
- new net D-: R2.2, U2.3 (D-)
- new net GND: C1.2, C2.2, C3.2, C4.2, C5.2, C6.2, C7.2, C8.1, J1.6 (GND), R4.2, R5.2, R6.2, SW1.2, U1.1 (GND), U2.15 (GND), U2.23 (GND), U2.35 (GND), U2.43 (GND), U2.5 (UGND), USB1.1 (GND), USB1.12 (GND), USB1.13 (SHIELD), X1.2, X1.4
- new net MISO: J1.1 (MISO), U2.11 (PB3)
- new net MOSI: J1.4 (MOSI), U2.10 (PB2)
- new net RESET: J1.5 (~{RST}), R1.2, SW1.1, U2.13 (~{RESET})
- new net SCK: J1.3 (SCK), U2.9 (PB1)
- new net VCC: F1.1, U1.4 (VCC), USB1.11 (VBUS), USB1.2 (VBUS)
- new net XTAL1: C1.1, U2.17 (XTAL1), X1.1
- new net XTAL2: C2.1, U2.16 (XTAL2), X1.3
- new net col0: MX1.1 (COL)
- new net col1: MX2.1 (COL)
- new net col2: MX3.1 (COL)
- new net row0: D1.1 (K), D2.1 (K), D3.1 (K)
- no-connect marks 0 -> 27

Commit message: route pcb
Parts:
- C1, C2, C3, C4, C5, C6, C7, C8: footprint (none) -> Capacitor_SMD:C_0805_2012Metric_Pad1.18x1.45mm_HandSolder
- D1, D2, D3: footprint (none) -> Diode_SMD:D_SOD-123
- F1: footprint (none) -> Fuse:Fuse_1206_3216Metric_Pad1.42x1.75mm_HandSolder
- J1: footprint (none) -> random-keyboard-parts:Reset_Pretty-Mask
- MX1, MX2, MX3: footprint (none) -> MX_Only:MXOnly-1U-Hotswap
- R1, R2, R3, R4, R5, R6: footprint (none) -> Resistor_SMD:R_0805_2012Metric_Pad1.20x1.40mm_HandSolder
- SW1: footprint (none) -> Button_Switch_SMD:SW_SPST_SKQG_WithStem
- U1: footprint (none) -> random-keyboard-parts:SOT143B
- USB1: footprint (none) -> Type-C:HRO-TYPE-C-31-M-12-HandSoldering
- X1: footprint (none) -> Crystal:Crystal_SMD_3225-4Pin_3.2x2.5mm_HandSoldering
Connections:
- net col0: now also U2.41 (PF0)
- net col1: now also U2.39 (PF4)
- net col2: now also U2.38 (PF5)
- net row0: now also U2.40 (PF1)
- net DN: now reaches R2.1, U1.3 (IO2), USB1.5 (DN2), USB1.7 (DN1)
- net DP: now reaches R3.1, U1.2 (IO1), USB1.6 (DP1), USB1.8 (DP2)
- no-connect marks 27 -> 23

Commit message: antishear bois
Parts:
- MX1, MX2, MX3: footprint MX_Only:MXOnly-1U-Hotswap -> MX_Only:MXOnly-1U-Hotswap-Antishear
Changed lines of the file:
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@@
       (effects (font (size 0.508 0.508)))
     )
-    (property "Footprint" "MX_Only:MXOnly-1U-Hotswap" (id 2) (at 211.455 92.075 0)
+    (property "Footprint" "MX_Only:MXOnly-1U-Hotswap-Antishear" (id 2) (at 211.455 92.075 0)
       (effects (font (size 1.524 1.524)) hide)
     )
@@
       (effects (font (size 0.508 0.508)))
     )
-    (property "Footprint" "MX_Only:MXOnly-1U-Hotswap" (id 2) (at 234.315 92.075 0)
+    (property "Footprint" "MX_Only:MXOnly-1U-Hotswap-Antishear" (id 2) (at 234.315 92.075 0)
       (effects (font (size 1.524 1.524)) hide)
     )
@@
       (effects (font (size 0.508 0.508)))
     )
-    (property "Footprint" "MX_Only:MXOnly-1U-Hotswap" (id 2) (at 222.885 92.075 0)
+    (property "Footprint" "MX_Only:MXOnly-1U-Hotswap-Antishear" (id 2) (at 222.885 92.075 0)
       (effects (font (size 1.524 1.524)) hide)
     )
@@
     )
     (path "/0bfe75c1-05d0-4adc-9dc7-2df1c3471385"
-      (reference "MX1") (unit 1) (value "Z") (footprint "MX_Only:MXOnly-1U-Hotswap")
+      (reference "MX1") (unit 1) (value "Z") (footprint "MX_Only:MXOnly-1U-Hotswap-Antishear")
     )
     (path "/d821d36c-8203-4138-be12-eaf5cc3caaee"
-      (reference "MX2") (unit 1) (value "X") (footprint "MX_Only:MXOnly-1U-Hotswap")
+      (reference "MX2") (unit 1) (value "X") (footprint "MX_Only:MXOnly-1U-Hotswap-Antishear")
     )
     (path "/b1de568c-5426-4aff-a66a-482e948a724a"
-      (reference "MX3") (unit 1) (value "C") (footprint "MX_Only:MXOnly-1U-Hotswap")
+      (reference "MX3") (unit 1) (value "C") (footprint "MX_Only:MXOnly-1U-Hotswap-Antishear")
     )
     (path "/5bf3412a-aefc-4123-9a7d-157d90836c07"
